File: rf_module/rf_module.kicad_sch (KiCad schematic)
At the start: 68 parts, among them J1 Conn_01x14, J2 UHF, Q1 SQ2318, U1 LP2985-1.8, U2 TYKTBCSANF-26.000000, U3 NL17SV04XV5T2G, U4 Si4463, U5 TQP3M9036, U6 LFCG-490+, U7 F2972

Commit message: feat: minor schematic adjustments and pcb layout
Parts:
- added H1, H2, H3, H4: MH, MountingHole:MountingHole_2.2mm_M2_Pad_Via, symbol Mechanical:MountingHole_Pad
- J2: footprint Connector_Coaxial:SMB_Jack_Vertical -> Connector_Coaxial:SMA_Amphenol_132134_Vertical
- U7: footprint Package_DFN_QFN:IDT_NEG12_1EP_2x2mm_P0.5mm_EP1.1x1.1mm_ThermalVias -> lsf-kicad-lib:IDT_NEG-12-1EP_2x2mm_P0.5mm_EP1.1x1.1mm_ThermalVias
Connections:
- net GND: now also H1.1, H2.1, H3.1, H4.1
- net PA_Fault: now also J1.4 (Pin_4); no longer J1.13 (Pin_13)
- net Si4463_GPIO0: now also J1.9 (Pin_9); no longer J1.4 (Pin_4)
- net Si4463_GPIO1: now also J1.10 (Pin_10); no longer J1.5 (Pin_5)
- net Si4463_SDI: now also J1.12 (Pin_12); no longer J1.8 (Pin_8)
- net Si4463_SDO: now also J1.13 (Pin_13); no longer J1.9 (Pin_9)
- net Si4463_SPI_CLK: now also J1.11 (Pin_11); no longer J1.7 (Pin_7)
- net Si4463_nIRQ: now also J1.8 (Pin_8); no longer J1.11 (Pin_11)
- net Si4463_nSEL: now also J1.7 (Pin_7); no longer J1.10 (Pin_10)
- net TX_Block: now also J1.5 (Pin_5); no longer J1.12 (Pin_12)
- net 3V3_Si_Filt: now reaches C15.1, R6.1, U4.8 (VDD)
- net RF_Si_Out: now reaches C17.1, L8.1, U4.4 (TX)
- net RF_Si_Inp: now reaches C20.1, L10.1, L9.1, U4.2 (RXp)
- net RF_Si_Inn: now reaches C22.1, L9.2, U4.3 (RXn)
- net RF_LPF1_Mid2: now reaches C4.1, L2.2, L3.1
- net RF_Sw2: now reaches U6.4 (OUT), U7.11 (RF2)
- net RF_Sw: now reaches C32.1, U7.2 (RFC)
- net RF_Sw1: now reaches C28.2, C29.1, L14.2, U7.5 (RF1)
- net RF_BPF2_Out: now reaches C22.2, C7.1, L10.2, L4.2, L5.1
- net RF_BPF2_Mid: now reaches C10.1, L5.2
- net RF_BPF2_In: now reaches C10.2, C11.1, C12.1, L6.2
- net RF_Si_Match: now reaches C17.2, L12.1
- net RF_LPF1_In: now reaches C26.1, L1.1, L12.2
- net RF_BPF1_Mid: now reaches C28.1, L13.2
- net RF_Connector: now reaches C32.2, J2.1 (In)
- net RF_BPF1_Out: now reaches C18.2, C24.1, L11.2, L13.1
- net RF_LNA_Out: now reaches C12.2, L7.1, U5.7 (RFOUT)
- net RF_LNA_In: now reaches C18.1, U5.2 (RFIN)
- net RF_LPF1_Mid1: now reaches C2.1, L1.2, L2.1
- net UHF_PA/RF_IN renamed RF_LPF1_Out
- net UHF_PA/RF_OUT renamed RF_LPF2_In
Other:
- sheet UHF_PA ports: added PA_Fault; removed PA_FAULT
- moved on the sheet: C32

Commit message: feat: implement LNA activation on RX and PA_Enable in schematic (layout TODO)
Parts:
- removed J1: Conn_01x14, Connector_PinHeader_2.54mm:PinHeader_1x14_P2.54mm_Vertical, symbol Connector_Generic:Conn_01x14
- added C46: 100p, Capacitor_SMD:C_0402_1005Metric, symbol Device:C_Small
- added J1: Conn_01x15, Connector_PinHeader_2.54mm:PinHeader_1x15_P2.54mm_Vertical, symbol Connector_Generic:Conn_01x15
- added Q2, Q3: SQ2318, Package_TO_SOT_SMD:SOT-23, symbol Device:Q_NMOS_GSD
- added R11, R16: 100, Resistor_SMD:R_0603_1608Metric, symbol Device:R
- added R14, R15: 10k, Resistor_SMD:R_0603_1608Metric, symbol Device:R_Small
- added TP6: RX_Active, TestPoint:TestPoint_Pad_D2.5mm, symbol Connector:TestPoint
- added U10: NL17SV04XV5T2G, Package_TO_SOT_SMD:SOT-553, symbol 74xGxx:74LVC1GU04DRL
- R8: value 10k -> 100; Mnf. Vishay -> (none); PartNumber CRCW040210K0FKEDC -> CR0402-FX-3302GLF
Connections:
- net +3V3: now also C46.1, J1.2 (Pin_2), U10.5 (VCC)
- net +5V: now also J1.1 (Pin_1)
- net GND: now also C46.2, J1.15 (Pin_15), J1.3 (Pin_3), Q2.2 (S), Q3.2 (S), R14.1, R15.1, U10.3 (GND); no longer R8.2
- net PA_Fault: now also J1.4 (Pin_4)
- net Si4463_GPIO0: now also J1.10 (Pin_10)
- net Si4463_GPIO1: now also J1.11 (Pin_11)
- net Si4463_SDI: now also J1.13 (Pin_13)
- net Si4463_SDN: now also J1.7 (Pin_7)
- net Si4463_SDO: now also J1.14 (Pin_14)
- net Si4463_SPI_CLK: now also J1.12 (Pin_12)
- net Si4463_nIRQ: now also J1.9 (Pin_9)
- net Si4463_nSEL: now also J1.8 (Pin_8)
- net TX_Active: no longer R7.2
- net RX_Active: now reaches U4.19 (GPIO2)
- net RX_Active: now also TP6.1, U10.2
- net at R4.2, R5.2, U3.2: now also R8.2
- net at R7.1, U5.6 (Shut_Down): no longer R8.1
- net TX_Block renamed PA_Block
- net PA_Block: now also J1.6 (Pin_6)
- new net: Q2.1 (G), R11.2, R14.2
- new net: Q3.1 (G), R15.2, R16.2
- new net: Q3.3 (D), R11.1
- new net: R7.2, U10.4
- new net: Q2.3 (D), R8.1
- new net PA_Enable: J1.5 (Pin_5), R16.1
- no-connect marks 3 -> 2
Other:
- moved on the sheet: C8, Q1, R2, R3, R4, R5, R7, TP2, U3

Commit message: fix: component values of TX PA input matching and filter
Parts:
- C2: value 12p -> 7.5p
- C4: value 10p -> 7.5p
- L1: value 30n -> 33n
- L2: value 36n -> 51n
- L3: value 22n -> 33n
Other:
- note removed: "Coilcraft 0402HP Series Inductors"
Changed lines of the file:
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@@
     (effects (font (size 1.27 1.27)) (justify left bottom))
   )
-  (text "Coilcraft 0402HP Series Inductors" (at 26.67 105.41 0)
-    (effects (font (size 1.27 1.27)) (justify left bottom))
-  )
   (label "Si4463_SPI_CLK" (at 101.6 78.74 0) (fields_autoplaced)
     (effects (font (size 1.27 1.27)) (justify left bottom))
@@
       (effects (font (size 1.27 1.27)) (justify right))
     )
-    (property "Value" "22n" (at 57.15 109.22 90)
+    (property "Value" "33n" (at 57.15 109.22 90)
       (effects (font (size 1.27 1.27)) (justify left))
     )
@@
       (effects (font (size 1.27 1.27)) (justify left))
     )
-    (property "Value" "10p" (at 52.07 120.65 0)
+    (property "Value" "7.5p" (at 52.07 120.65 0)
       (effects (font (size 1.27 1.27)) (justify left))
     )
@@
       (effects (font (size 1.27 1.27)) (justify left))
     )
-    (property "Value" "12p" (at 39.37 120.65 0)
+    (property "Value" "7.5p" (at 39.37 120.65 0)
       (effects (font (size 1.27 1.27)) (justify left))
     )
@@
       (effects (font (size 1.27 1.27)) (justify right))
     )
-    (property "Value" "36n" (at 44.45 109.22 90)
+    (property "Value" "51n" (at 44.45 109.22 90)
       (effects (font (size 1.27 1.27)) (justify left))
     )
@@
       (effects (font (size 1.27 1.27)) (justify right))
     )
-    (property "Value" "30n" (at 31.75 109.22 90)
+    (property "Value" "33n" (at 31.75 109.22 90)
       (effects (font (size 1.27 1.27)) (justify left))
     )
